Commit message: nav2: added mapping config

File: autocar_description/urdf/wl_rccar_v1.xacro (robot description, xacro)
@@ -59,5 +59,4 @@
                                 <origin xyz="0 0 0" rpy="0 0 0" />
                                 <geometry>
-                                        <!-- <mesh filename="package://autocar_description/meshes/wl_wheel.dae" /> -->
                                         <cylinder length="${wheel_length}" radius="${wheel_radius}" />
                                 </geometry>
